Commit message: Lab 4: Replace worksheet with complete solution (2-DoF + control package)
- URDF: complete 2-DoF manipulator with gazebo_ros_control plugin and transmissions
- Add ex_robot1_control package (YAML config + launch)
- Update README to solution-oriented documentation
- Keep TODO section markers for slide reference

File: src/ex_robot1_description/urdf/ex_robot1.urdf (robot description, URDF)
Before this commit: robot ex_robot1, 1 links, 0 joints
Links:
- added link link1, mass 3; collision box size=0.3 0.3 3; visual box size=0.3 0.3 3
- added link link2, mass 3; collision box size=0.3 0.3 3; visual box size=0.3 0.3 3
- added link world
Joints:
- added joint fixed: type fixed, parent world, child base_link, origin xyz=0 0 0.5 rpy=0 0 0
- added joint joint1: type continuous, parent base_link, child link1, origin xyz=0 0 0.5 rpy=0 0 0, axis 0 1 0
- added joint joint2: type continuous, parent link1, child link2, origin xyz=0 0 3 rpy=0 0 0, axis 0 1 0
